File: hardware/currentsensormodule.kicad_pcb (KiCad board)
At the start: 2 copper layers, 97.9 x 70.4 mm, 104 parts, among them J101 USART, J102 STLink, J103 Sensor1, J104 Sensor2, J105 RJ45, J106 RJ45, U101 LM324, U103 K78L15-1000R3, U104 K78L15-1000R3, U105 AMS1117-5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

Commit message: hardware: longer PCB design (main is wider)
Parts:
- moved C101 19.7 mm to (135.8, 77.6)
- moved J103 14.4 mm to (191.5, 118.6)
- moved J104 14.4 mm to (191.5, 92.5)
- moved H103 9.24 mm to (175.5, 73.7)
- moved H104 8.78 mm to (175.5, 125.9)
- moved J102 6.83 mm to (144.7, 76.5), turned to 90 degrees
- moved H102 6.35 mm to (98.0, 73.7)
- moved D106 6.12 mm to (145.8, 86.2)
- moved H101 5.66 mm to (98.0, 125.9)
- moved J101 2.50 mm to (158.9, 78.2), turned to 90 degrees
- moved C115 1.55 mm to (141.1, 73.7), turned to 0 degrees
Routing:
- net +15V: track 142.1 -> 162.3 mm
- net /Bipolar Analog/in1+: track 15.5 -> 30.3 mm
- net /Bipolar Analog/in2+: track 21.7 -> 36.4 mm
- net -15V: track 109.5 -> 124.0 mm
- net GND: track 112.3 -> 101.5 mm
- net +3V3: track 106.6 -> 98.1 mm
- net /STM32/USART1_RX: track 35.6 -> 29.9 mm
- net /STM32/SWDIO: track 28.1 -> 22.4 mm, vias 3 -> 1
- net /STM32/SWO: track 18.5 -> 13.5 mm
- net /STM32/USART1_TX: track 26.7 -> 31.0 mm
- net /STM32/RESET: track 29.8 -> 26.2 mm
- net Net-(D106-Pad2): track 5.34 -> 2.93 mm
Other:
- board outline removed
