File: hardware/analog_bipolar.kicad_sch (KiCad schematic)
At the start: 43 parts, among them U1 LM324

Commit message: Troca do atmega328p -> STM32F103C8T Já que tem CAN integrado e ADC 12 bits (ao invés de 10)
Parts:
- removed D2, D7, D9: 4V7, Diode_SMD:D_MiniMELF_Handsoldering, symbol Device:D_Zener_Small
- added D102, D103, D104: 3V9, Diode_SMD:D_MiniMELF_Handsoldering, symbol Device:D_Zener_Small
- C102: renamed from C10; footprint Capacitor_SMD:C_0805_2012Metric_Pad1.18x1.45mm_HandSolder -> (none)
- C103: renamed from C29; footprint Capacitor_SMD:C_0805_2012Metric_Pad1.18x1.45mm_HandSolder -> (none)
- C104: renamed from C11; footprint Capacitor_SMD:C_0805_2012Metric_Pad1.18x1.45mm_HandSolder -> (none)
- C105: renamed from C30; footprint Capacitor_SMD:C_0805_2012Metric_Pad1.18x1.45mm_HandSolder -> (none)
- C106: renamed from C12; footprint Capacitor_SMD:C_0805_2012Metric_Pad1.18x1.45mm_HandSolder -> (none)
- C107: renamed from C31; footprint Capacitor_SMD:C_0805_2012Metric_Pad1.18x1.45mm_HandSolder -> (none)
- C108: renamed from C13; footprint Capacitor_SMD:C_0805_2012Metric_Pad1.18x1.45mm_HandSolder -> (none)
- C109: renamed from C7; footprint Capacitor_SMD:C_0805_2012Metric_Pad1.18x1.45mm_HandSolder -> (none)
- D101: renamed from D8; value 4V7 -> (none); footprint Diode_SMD:D_MiniMELF_Handsoldering -> (none)
- R101: renamed from R2; footprint Resistor_SMD:R_0805_2012Metric_Pad1.20x1.40mm_HandSolder -> (none)
- R102: renamed from R19; footprint Resistor_SMD:R_0805_2012Metric_Pad1.20x1.40mm_HandSolder -> (none)
- R103: renamed from R3; footprint Resistor_SMD:R_0805_2012Metric_Pad1.20x1.40mm_HandSolder -> (none)
- R104: renamed from R4; footprint Resistor_SMD:R_0805_2012Metric_Pad1.20x1.40mm_HandSolder -> (none)
- R105: renamed from R20; footprint Resistor_SMD:R_0805_2012Metric_Pad1.20x1.40mm_HandSolder -> (none)
- R106: renamed from R21; footprint Resistor_SMD:R_0805_2012Metric_Pad1.20x1.40mm_HandSolder -> (none)
- R107: renamed from R5; footprint Resistor_SMD:R_0805_2012Metric_Pad1.20x1.40mm_HandSolder -> (none)
- R108: renamed from R6; footprint Resistor_SMD:R_0805_2012Metric_Pad1.20x1.40mm_HandSolder -> (none)
- R109: renamed from R22; footprint Resistor_SMD:R_0805_2012Metric_Pad1.20x1.40mm_HandSolder -> (none)
- R110: renamed from R23; footprint Resistor_SMD:R_0805_2012Metric_Pad1.20x1.40mm_HandSolder -> (none)
- R111: renamed from R7; footprint Resistor_SMD:R_0805_2012Metric_Pad1.20x1.40mm_HandSolder -> (none)
- R112: renamed from R24; footprint Resistor_SMD:R_0805_2012Metric_Pad1.20x1.40mm_HandSolder -> (none)
- R113: renamed from R8; footprint Resistor_SMD:R_0805_2012Metric_Pad1.20x1.40mm_HandSolder -> (none)
- R114: renamed from R25; footprint Resistor_SMD:R_0805_2012Metric_Pad1.20x1.40mm_HandSolder -> (none)
- R115: renamed from R9; footprint Resistor_SMD:R_0805_2012Metric_Pad1.20x1.40mm_HandSolder -> (none)
- R116: renamed from R26; footprint Resistor_SMD:R_0805_2012Metric_Pad1.20x1.40mm_HandSolder -> (none)
- R117: renamed from R27; footprint Resistor_SMD:R_0805_2012Metric_Pad1.20x1.40mm_HandSolder -> (none)
- R118: renamed from R28; footprint Resistor_SMD:R_0805_2012Metric_Pad1.20x1.40mm_HandSolder -> (none)
- renumbered TP2 to TP101, TP18 to TP102, TP3 to TP103, TP4 to TP104, TP19 to TP105, TP20 to TP106, TP5 to TP107, TP21 to TP108, TP6 to TP109, TP22 to TP110, TP7 to TP111, TP23 to TP112, U1 to U101
Connections:
- net GND: now also D102.2 (A), D104.2 (A)
- net out1: now also D102.1 (K)
- net out2: now also D103.2 (A), D104.1 (K)
- net +5V renamed +3V3
- net +3V3: now also D103.1 (K)
Other:
- moved on the sheet: C108, C109, U101E

Commit message: Primeiro protótipo da PCB
Parts:
- C102, C103, C104, C105, C106, C107, C108, C109: footprint (none) -> Capacitor_SMD:C_0603_1608Metric_Pad1.08x0.95mm_HandSolder
- D101: value (none) -> 3V9; footprint (none) -> Diode_SMD:D_MiniMELF_Handsoldering
- R101, R102, R103, R104, R105, R106, R107, R108, R109, R110, R111, R112, R113, R114, R115, R116, R117, R118: footprint (none) -> Resistor_SMD:R_0603_1608Metric_Pad0.98x0.95mm_HandSolder
Changed lines of the file:
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@@
       (effects (font (size 1.27 1.27)) (justify left))
     )
-    (property "Footprint" "" (id 2) (at 100.33 67.31 0)
+    (property "Footprint" "Resistor_SMD:R_0603_1608Metric_Pad0.98x0.95mm_HandSolder" (id 2) (at 100.33 67.31 0)
       (effects (font (size 1.27 1.27)) hide)
     )
@@
       (effects (font (size 1.27 1.27)) (justify left))
     )
-    (property "Footprint" "" (id 2) (at 100.33 72.39 0)
+    (property "Footprint" "Resistor_SMD:R_0603_1608Metric_Pad0.98x0.95mm_HandSolder" (id 2) (at 100.33 72.39 0)
       (effects (font (size 1.27 1.27)) hide)
     )
@@
       (effects (font (size 1.27 1.27)) (justify left))
     )
-    (property "Footprint" "" (id 2) (at 144.78 69.85 0)
+    (property "Footprint" "Resistor_SMD:R_0603_1608Metric_Pad0.98x0.95mm_HandSolder" (id 2) (at 144.78 69.85 0)
       (effects (font (size 1.27 1.27)) hide)
     )
@@
       (effects (font (size 1.27 1.27)) (justify left))
     )
-    (property "Footprint" "" (id 2) (at 154.94 69.85 0)
+    (property "Footprint" "Resistor_SMD:R_0603_1608Metric_Pad0.98x0.95mm_HandSolder" (id 2) (at 154.94 69.85 0)
       (effects (font (size 1.27 1.27)) hide)
     )
@@
       (effects (font (size 1.27 1.27)) (justify left))
     )
-    (property "Footprint" "" (id 2) (at 160.02 76.2 0)
+    (property "Footprint" "Capacitor_SMD:C_0603_1608Metric_Pad1.08x0.95mm_HandSolder" (id 2) (at 160.02 76.2 0)
       (effects (font (size 1.27 1.27)) hide)
     )
@@
       (effects (font (size 1.27 1.27)) (justify left))
     )
-    (property "Footprint" "" (id 2) (at 149.86 76.2 0)
+    (property "Footprint" "Capacitor_SMD:C_0603_1608Metric_Pad1.08x0.95mm_HandSolder" (id 2) (at 149.86 76.2 0)
       (effects (font (size 1.27 1.27)) hide)
     )
@@
       (effects (font (size 1.27 1.27)) (justify left))
     )
-    (property "Footprint" "" (id 2) (at 118.11 60.96 0)
+    (property "Footprint" "Resistor_SMD:R_0603_1608Metric_Pad0.98x0.95mm_HandSolder" (id 2) (at 118.11 60.96 0)
       (effects (font (size 1.27 1.27)) hide)
     )
@@
       (effects (font (size 1.27 1.27)) (justify left))
     )
-    (property "Footprint" "" (id 2) (at 118.11 78.74 0)
+    (property "Footprint" "Resistor_SMD:R_0603_1608Metric_Pad0.98x0.95mm_HandSolder" (id 2) (at 118.11 78.74 0)
       (effects (font (size 1.27 1.27)) hide)
     )
@@
       (effects (font (size 1.27 1.27)) (justify left))
     )
-    (property "Footprint" "" (id 2) (at 87.63 69.85 0)
+    (property "Footprint" "Resistor_SMD:R_0603_1608Metric_Pad0.98x0.95mm_HandSolder" (id 2) (at 87.63 69.85 0)
       (effects (font (size 1.27 1.27)) hide)
     )
@@
       (effects (font (size 1.27 1.27)) (justify left))
     )
-    (property "Footprint" "" (id 2) (at 134.62 69.85 0)
+    (property "Footprint" "Resistor_SMD:R_0603_1608Metric_Pad0.98x0.95mm_HandSolder" (id 2) (at 134.62 69.85 0)
       (effects (font (size 1.27 1.27)) hide)
     )
@@
       (effects (font (size 1.27 1.27)) (justify left))
     )
-    (property "Footprint" "" (id 2) (at 139.7 76.2 0)
+    (property "Footprint" "Capacitor_SMD:C_0603_1608Metric_Pad1.08x0.95mm_HandSolder" (id 2) (at 139.7 76.2 0)
       (effects (font (size 1.27 1.27)) hide)
     )
@@
       (effects (font (size 1.27 1.27)) (justify left))
     )
-    (property "Footprint" "" (id 2) (at 232.41 102.87 0)
+    (property "Footprint" "Capacitor_SMD:C_0603_1608Metric_Pad1.08x0.95mm_HandSolder" (id 2) (at 232.41 102.87 0)
       (effects (font (size 1.27 1.27)) hide)
     )
@@
     (in_bom yes) (on_board yes)
     (property "Reference" "D101" (id 0) (at 199.136 59.69 0))
-    (property "Value" "" (id 1) (at 194.564 59.69 0))
-    (property "Footprint" "" (id 2) (at 196.85 59.69 90)
+    (property "Value" "3V9" (id 1) (at 194.564 59.69 0))
+    (property "Footprint" "Diode_SMD:D_MiniMELF_Handsoldering" (id 2) (at 196.85 59.69 90)
       (effects (font (size 1.27 1.27)) hide)
     )
@@
       (effects (font (size 1.27 1.27)) (justify left))
     )
-    (property "Footprint" "" (id 2) (at 166.37 76.2 0)
+    (property "Footprint" "Resistor_SMD:R_0603_1608Metric_Pad0.98x0.95mm_HandSolder" (id 2) (at 166.37 76.2 0)
       (effects (font (size 1.27 1.27)) hide)
     )
@@
       (effects (font (size 1.27 1.27)) (justify left))
     )
-    (property "Footprint" "" (id 2) (at 232.41 113.03 0)
+    (property "Footprint" "Capacitor_SMD:C_0603_1608Metric_Pad1.08x0.95mm_HandSolder" (id 2) (at 232.41 113.03 0)
       (effects (font (size 1.27 1.27)) hide)
     )
@@
       (effects (font (size 1.27 1.27)) (justify left))
     )
-    (property "Footprint" "" (id 2) (at 101.6 114.3 0)
+    (property "Footprint" "Resistor_SMD:R_0603_1608Metric_Pad0.98x0.95mm_HandSolder" (id 2) (at 101.6 114.3 0)
       (effects (font (size 1.27 1.27)) hide)
     )
@@
       (effects (font (size 1.27 1.27)) (justify left))
     )
-    (property "Footprint" "" (id 2) (at 101.6 119.38 0)
+    (property "Footprint" "Resistor_SMD:R_0603_1608Metric_Pad0.98x0.95mm_HandSolder" (id 2) (at 101.6 119.38 0)
       (effects (font (size 1.27 1.27)) hide)
     )
@@
       (effects (font (size 1.27 1.27)) (justify left))
     )
-    (property "Footprint" "" (id 2) (at 146.05 116.84 0)
+    (property "Footprint" "Resistor_SMD:R_0603_1608Metric_Pad0.98x0.95mm_HandSolder" (id 2) (at 146.05 116.84 0)
       (effects (font (size 1.27 1.27)) hide)
     )
@@
       (effects (font (size 1.27 1.27)) (justify left))
     )
-    (property "Footprint" "" (id 2) (at 156.21 116.84 0)
+    (property "Footprint" "Resistor_SMD:R_0603_1608Metric_Pad0.98x0.95mm_HandSolder" (id 2) (at 156.21 116.84 0)
       (effects (font (size 1.27 1.27)) hide)
     )
@@
       (effects (font (size 1.27 1.27)) (justify left))
     )
-    (property "Footprint" "" (id 2) (at 161.29 123.19 0)
+    (property "Footprint" "Capacitor_SMD:C_0603_1608Metric_Pad1.08x0.95mm_HandSolder" (id 2) (at 161.29 123.19 0)
       (effects (font (size 1.27 1.27)) hide)
     )
@@
       (effects (font (size 1.27 1.27)) (justify left))
     )
-    (property "Footprint" "" (id 2) (at 151.13 123.19 0)
+    (property "Footprint" "Capacitor_SMD:C_0603_1608Metric_Pad1.08x0.95mm_HandSolder" (id 2) (at 151.13 123.19 0)
       (effects (font (size 1.27 1.27)) hide)
     )
@@
       (effects (font (size 1.27 1.27)) (justify left))
     )
-    (property "Footprint" "" (id 2) (at 119.38 107.95 0)
+    (property "Footprint" "Resistor_SMD:R_0603_1608Metric_Pad0.98x0.95mm_HandSolder" (id 2) (at 119.38 107.95 0)
       (effects (font (size 1.27 1.27)) hide)
     )
@@
       (effects (font (size 1.27 1.27)) (justify left))
     )
-    (property "Footprint" "" (id 2) (at 119.38 125.73 0)
+    (property "Footprint" "Resistor_SMD:R_0603_1608Metric_Pad0.98x0.95mm_HandSolder" (id 2) (at 119.38 125.73 0)
       (effects (font (size 1.27 1.27)) hide)
     )
@@
       (effects (font (size 1.27 1.27)) (justify left))
     )
-    (property "Footprint" "" (id 2) (at 88.9 116.84 0)
+    (property "Footprint" "Resistor_SMD:R_0603_1608Metric_Pad0.98x0.95mm_HandSolder" (id 2) (at 88.9 116.84 0)
       (effects (font (size 1.27 1.27)) hide)
     )
@@
       (effects (font (size 1.27 1.27)) (justify left))
     )
-    (property "Footprint" "" (id 2) (at 135.89 116.84 0)
+    (property "Footprint" "Resistor_SMD:R_0603_1608Metric_Pad0.98x0.95mm_HandSolder" (id 2) (at 135.89 116.84 0)
       (effects (font (size 1.27 1.27)) hide)
     )
@@
       (effects (font (size 1.27 1.27)) (justify left))
     )
-    (property "Footprint" "" (id 2) (at 140.97 123.19 0)
+    (property "Footprint" "Capacitor_SMD:C_0603_1608Metric_Pad1.08x0.95mm_HandSolder" (id 2) (at 140.97 123.19 0)
       (effects (font (size 1.27 1.27)) hide)
     )
@@
       (effects (font (size 1.27 1.27)) (justify left))
     )
-    (property "Footprint" "" (id 2) (at 167.64 123.19 0)
+    (property "Footprint" "Resistor_SMD:R_0603_1608Metric_Pad0.98x0.95mm_HandSolder" (id 2) (at 167.64 123.19 0)
       (effects (font (size 1.27 1.27)) hide)
     )
@@
       (effects (font (size 1.27 1.27)) hide)
     )
-    (property "Value" "" (id 1) (at 196.85 49.7642 0))
+    (property "Value" "+3.3V" (id 1) (at 196.85 49.7642 0))
     (property "Footprint" "" (id 2) (at 196.85 53.34 0)
       (effects (font (size 1.27 1.27)) hide)

Commit message: STLink 3v3 protection diode, silkscreen updates
Parts:
- TP101: value in+ -> (none)
- TP102: value in+ -> (none); footprint TestPoint:TestPoint_Pad_2.0x2.0mm -> (none)
- TP103: value op_a_in- -> (none)
- TP104, TP106: value op_a_in+ -> (none); footprint TestPoint:TestPoint_Pad_2.0x2.0mm -> (none)
- TP105: value op_a_in- -> (none); footprint TestPoint:TestPoint_Pad_2.0x2.0mm -> (none)
- TP107, TP108: value op_a_out -> (none); footprint TestPoint:TestPoint_Pad_2.0x2.0mm -> (none)
- TP109, TP110: value op_b_in+ -> (none); footprint TestPoint:TestPoint_Pad_2.0x2.0mm -> (none)
- TP111, TP112: value op_b_out -> (none); footprint TestPoint:TestPoint_Pad_2.0x2.0mm -> (none)
Changed lines of the file:
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@@
       (effects (font (size 1.27 1.27)) (justify bottom))
     )
-    (property "Value" "op_a_out" (id 1) (at 128.27 53.34 0))
-    (property "Footprint" "TestPoint:TestPoint_Pad_2.0x2.0mm" (id 2) (at 128.27 59.69 0)
+    (property "Value" "" (id 1) (at 128.27 53.34 0))
+    (property "Footprint" "" (id 2) (at 128.27 59.69 0)
       (effects (font (size 1.27 1.27)) hide)
     )
@@
       (effects (font (size 1.27 1.27)) (justify bottom))
     )
-    (property "Value" "op_a_in-" (id 1) (at 107.95 53.34 0))
+    (property "Value" "" (id 1) (at 107.95 53.34 0))
     (property "Footprint" "TestPoint:TestPoint_Pad_2.0x2.0mm" (id 2) (at 107.95 59.69 0)
       (effects (font (size 1.27 1.27)) hide)
@@
       (effects (font (size 1.27 1.27)) (justify bottom))
     )
-    (property "Value" "op_a_in+" (id 1) (at 107.95 86.36 0))
-    (property "Footprint" "TestPoint:TestPoint_Pad_2.0x2.0mm" (id 2) (at 107.95 80.01 0)
+    (property "Value" "" (id 1) (at 107.95 86.36 0))
+    (property "Footprint" "" (id 2) (at 107.95 80.01 0)
       (effects (font (size 1.27 1.27)) hide)
     )
@@
       (effects (font (size 1.27 1.27)) (justify bottom))
     )
-    (property "Value" "op_b_out" (id 1) (at 203.2 59.69 0))
-    (property "Footprint" "TestPoint:TestPoint_Pad_2.0x2.0mm" (id 2) (at 203.2 66.04 0)
+    (property "Value" "" (id 1) (at 203.2 59.69 0))
+    (property "Footprint" "" (id 2) (at 203.2 66.04 0)
       (effects (font (size 1.27 1.27)) hide)
     )
@@
       (effects (font (size 1.27 1.27)) (justify bottom))
     )
-    (property "Value" "op_b_in+" (id 1) (at 158.75 62.23 0))
-    (property "Footprint" "TestPoint:TestPoint_Pad_2.0x2.0mm" (id 2) (at 160.02 68.58 0)
+    (property "Value" "" (id 1) (at 158.75 62.23 0))
+    (property "Footprint" "" (id 2) (at 160.02 68.58 0)
       (effects (font (size 1.27 1.27)) hide)
     )
@@
       (effects (font (size 1.27 1.27)) (justify bottom))
     )
-    (property "Value" "in+" (id 1) (at 87.63 81.28 0))
+    (property "Value" "" (id 1) (at 87.63 81.28 0))
     (property "Footprint" "TestPoint:TestPoint_Pad_2.0x2.0mm" (id 2) (at 87.63 74.93 0)
       (effects (font (size 1.27 1.27)) hide)
@@
       (effects (font (size 1.27 1.27)) (justify bottom))
     )
-    (property "Value" "op_a_out" (id 1) (at 129.54 100.33 0))
-    (property "Footprint" "TestPoint:TestPoint_Pad_2.0x2.0mm" (id 2) (at 129.54 106.68 0)
+    (property "Value" "" (id 1) (at 129.54 100.33 0))
+    (property "Footprint" "" (id 2) (at 129.54 106.68 0)
       (effects (font (size 1.27 1.27)) hide)
     )
@@
       (effects (font (size 1.27 1.27)) (justify bottom))
     )
-    (property "Value" "op_a_in-" (id 1) (at 109.22 100.33 0))
-    (property "Footprint" "TestPoint:TestPoint_Pad_2.0x2.0mm" (id 2) (at 109.22 106.68 0)
+    (property "Value" "" (id 1) (at 109.22 100.33 0))
+    (property "Footprint" "" (id 2) (at 109.22 106.68 0)
       (effects (font (size 1.27 1.27)) hide)
     )
@@
       (effects (font (size 1.27 1.27)) (justify bottom))
     )
-    (property "Value" "op_a_in+" (id 1) (at 109.22 133.35 0))
-    (property "Footprint" "TestPoint:TestPoint_Pad_2.0x2.0mm" (id 2) (at 109.22 127 0)
+    (property "Value" "" (id 1) (at 109.22 133.35 0))
+    (property "Footprint" "" (id 2) (at 109.22 127 0)
       (effects (font (size 1.27 1.27)) hide)
     )
@@
       (effects (font (size 1.27 1.27)) (justify bottom))
     )
-    (property "Value" "op_b_out" (id 1) (at 204.47 106.68 0))
-    (property "Footprint" "TestPoint:TestPoint_Pad_2.0x2.0mm" (id 2) (at 204.47 113.03 0)
+    (property "Value" "" (id 1) (at 204.47 106.68 0))
+    (property "Footprint" "" (id 2) (at 204.47 113.03 0)
       (effects (font (size 1.27 1.27)) hide)
     )
@@
       (effects (font (size 1.27 1.27)) (justify bottom))
     )
-    (property "Value" "op_b_in+" (id 1) (at 160.02 109.22 0))
-    (property "Footprint" "TestPoint:TestPoint_Pad_2.0x2.0mm" (id 2) (at 161.29 115.57 0)
+    (property "Value" "" (id 1) (at 160.02 109.22 0))
+    (property "Footprint" "" (id 2) (at 161.29 115.57 0)
       (effects (font (size 1.27 1.27)) hide)
     )
@@
       (effects (font (size 1.27 1.27)) (justify bottom))
     )
-    (property "Value" "in+" (id 1) (at 88.9 128.27 0))
-    (property "Footprint" "TestPoint:TestPoint_Pad_2.0x2.0mm" (id 2) (at 88.9 121.92 0)
-      (effects (font (size 1.27 1.27)) hide)
-    )
+    (property "Value" "" (id 1) (at 88.9 128.27 0))
+    (property "Footprint" "" (id 2) (at 88.9 121.92 0)
+      (effects (font (size 1.27 1.27)) hide)
+    )

Commit message: Silkscreen finished, module components '.csv'
Parts:
- TP101: value (none) -> in+1
- TP102: value (none) -> in+2; footprint (none) -> TestPoint:TestPoint_Pad_2.0x2.0mm
- TP103: value (none) -> op_a_in-1
- TP104: value (none) -> op_a_in+1; footprint (none) -> TestPoint:TestPoint_Pad_2.0x2.0mm
- TP105: value (none) -> op_a_in-2; footprint (none) -> TestPoint:TestPoint_Pad_2.0x2.0mm
- TP106: value (none) -> op_a_in+2; footprint (none) -> TestPoint:TestPoint_Pad_2.0x2.0mm
- TP107: value (none) -> op_a_out1; footprint (none) -> TestPoint:TestPoint_Pad_2.0x2.0mm
- TP108: value (none) -> op_a_out2; footprint (none) -> TestPoint:TestPoint_Pad_2.0x2.0mm
- TP109: value (none) -> op_b_in+1; footprint (none) -> TestPoint:TestPoint_Pad_2.0x2.0mm
- TP110: value (none) -> op_b_in+2; footprint (none) -> TestPoint:TestPoint_Pad_2.0x2.0mm
- TP111: value (none) -> op_b_out1; footprint (none) -> TestPoint:TestPoint_Pad_2.0x2.0mm
- TP112: value (none) -> op_b_out2; footprint (none) -> TestPoint:TestPoint_Pad_2.0x2.0mm
Changed lines of the file:
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@@
       (effects (font (size 1.27 1.27)) (justify bottom))
     )
-    (property "Value" "" (id 1) (at 128.27 53.34 0))
-    (property "Footprint" "" (id 2) (at 128.27 59.69 0)
+    (property "Value" "op_a_out1" (id 1) (at 128.27 53.34 0))
+    (property "Footprint" "TestPoint:TestPoint_Pad_2.0x2.0mm" (id 2) (at 128.27 59.69 0)
       (effects (font (size 1.27 1.27)) hide)
     )
@@
       (effects (font (size 1.27 1.27)) (justify bottom))
     )
-    (property "Value" "" (id 1) (at 107.95 53.34 0))
+    (property "Value" "op_a_in-1" (id 1) (at 107.95 53.34 0))
     (property "Footprint" "TestPoint:TestPoint_Pad_2.0x2.0mm" (id 2) (at 107.95 59.69 0)
       (effects (font (size 1.27 1.27)) hide)
@@
       (effects (font (size 1.27 1.27)) (justify bottom))
     )
-    (property "Value" "" (id 1) (at 107.95 86.36 0))
-    (property "Footprint" "" (id 2) (at 107.95 80.01 0)
+    (property "Value" "op_a_in+1" (id 1) (at 107.95 86.36 0))
+    (property "Footprint" "TestPoint:TestPoint_Pad_2.0x2.0mm" (id 2) (at 107.95 80.01 0)
       (effects (font (size 1.27 1.27)) hide)
     )
@@
       (effects (font (size 1.27 1.27)) (justify bottom))
     )
-    (property "Value" "" (id 1) (at 203.2 59.69 0))
-    (property "Footprint" "" (id 2) (at 203.2 66.04 0)
+    (property "Value" "op_b_out1" (id 1) (at 203.2 59.69 0))
+    (property "Footprint" "TestPoint:TestPoint_Pad_2.0x2.0mm" (id 2) (at 203.2 66.04 0)
       (effects (font (size 1.27 1.27)) hide)
     )
@@
       (effects (font (size 1.27 1.27)) (justify bottom))
     )
-    (property "Value" "" (id 1) (at 158.75 62.23 0))
-    (property "Footprint" "" (id 2) (at 160.02 68.58 0)
+    (property "Value" "op_b_in+1" (id 1) (at 158.75 62.23 0))
+    (property "Footprint" "TestPoint:TestPoint_Pad_2.0x2.0mm" (id 2) (at 160.02 68.58 0)
       (effects (font (size 1.27 1.27)) hide)
     )
@@
       (effects (font (size 1.27 1.27)) (justify bottom))
     )
-    (property "Value" "" (id 1) (at 87.63 81.28 0))
+    (property "Value" "in+1" (id 1) (at 87.63 81.28 0))
     (property "Footprint" "TestPoint:TestPoint_Pad_2.0x2.0mm" (id 2) (at 87.63 74.93 0)
       (effects (font (size 1.27 1.27)) hide)
@@
       (effects (font (size 1.27 1.27)) (justify bottom))
     )
-    (property "Value" "" (id 1) (at 129.54 100.33 0))
-    (property "Footprint" "" (id 2) (at 129.54 106.68 0)
+    (property "Value" "op_a_out2" (id 1) (at 129.54 100.33 0))
+    (property "Footprint" "TestPoint:TestPoint_Pad_2.0x2.0mm" (id 2) (at 129.54 106.68 0)
       (effects (font (size 1.27 1.27)) hide)
     )
@@
       (effects (font (size 1.27 1.27)) (justify bottom))
     )
-    (property "Value" "" (id 1) (at 109.22 100.33 0))
-    (property "Footprint" "" (id 2) (at 109.22 106.68 0)
+    (property "Value" "op_a_in-2" (id 1) (at 109.22 100.33 0))
+    (property "Footprint" "TestPoint:TestPoint_Pad_2.0x2.0mm" (id 2) (at 109.22 106.68 0)
       (effects (font (size 1.27 1.27)) hide)
     )
@@
       (effects (font (size 1.27 1.27)) (justify bottom))
     )
-    (property "Value" "" (id 1) (at 109.22 133.35 0))
-    (property "Footprint" "" (id 2) (at 109.22 127 0)
+    (property "Value" "op_a_in+2" (id 1) (at 109.22 133.35 0))
+    (property "Footprint" "TestPoint:TestPoint_Pad_2.0x2.0mm" (id 2) (at 109.22 127 0)
       (effects (font (size 1.27 1.27)) hide)
     )
@@
       (effects (font (size 1.27 1.27)) (justify bottom))
     )
-    (property "Value" "" (id 1) (at 204.47 106.68 0))
-    (property "Footprint" "" (id 2) (at 204.47 113.03 0)
+    (property "Value" "op_b_out2" (id 1) (at 204.47 106.68 0))
+    (property "Footprint" "TestPoint:TestPoint_Pad_2.0x2.0mm" (id 2) (at 204.47 113.03 0)
       (effects (font (size 1.27 1.27)) hide)
     )
@@
       (effects (font (size 1.27 1.27)) (justify bottom))
     )
-    (property "Value" "" (id 1) (at 160.02 109.22 0))
-    (property "Footprint" "" (id 2) (at 161.29 115.57 0)
+    (property "Value" "op_b_in+2" (id 1) (at 160.02 109.22 0))
+    (property "Footprint" "TestPoint:TestPoint_Pad_2.0x2.0mm" (id 2) (at 161.29 115.57 0)
       (effects (font (size 1.27 1.27)) hide)
     )
@@
       (effects (font (size 1.27 1.27)) (justify bottom))
     )
-    (property "Value" "" (id 1) (at 88.9 128.27 0))
-    (property "Footprint" "" (id 2) (at 88.9 121.92 0)
-      (effects (font (size 1.27 1.27)) hide)
-    )
+    (property "Value" "in+2" (id 1) (at 88.9 128.27 0))
+    (property "Footprint" "TestPoint:TestPoint_Pad_2.0x2.0mm" (id 2) (at 88.9 121.92 0)
+      (effects (font (size 1.27 1.27)) hide)
+    )
